Commit message: Improved camera parameters and documentation. Improved gazebo test world. Flipped the CAD normals.

File: urdf/camera.urdf.xacro (robot description, xacro)
@@ -1,55 +1,63 @@
 <?xml version="1.0" ?>
 <robot name="camera_projection_mapping" xmlns:xacro="http://ros.org/wiki/xacro">
-		<link name="camera_link">
-			<visual>
-				<origin xyz="0 0 0" rpy="0 0 0" />
-				<geometry>
-					<box size="0.2 0.1 0.4" />
-				</geometry>
-			</visual>
-			<inertial>
-				<mass value="1" />
-				<origin xyz="0 0 0" />
-				<inertia ixx="0.1" ixy="0.0" ixz="0.0" iyy="0.1" iyz="0.0" izz="0.1" />
-			</inertial>
-		</link>
-		<gazebo>
-			<static>true</static>
-		</gazebo>
-		<gazebo reference="camera_link">
-			<material>Gazebo/Blue</material>
-			<sensor type="camera" name="virtual_camera">
-				<camera name="projector_head">
-					<horizontal_fov>0.6859</horizontal_fov>
-					<image>
-						<width>1920</width>
-						<height>1080</height>
-						<format>R8G8B8</format>
-					</image>
-					<clip>
-						<near>0.02</near>
-						<far>300</far>
-					</clip>
-					<noise>
-						<type>gaussian</type>
-						<mean>0.0</mean>
-						<stddev>0.007</stddev>
-					</noise>
-				</camera>
-				<plugin name="camera_controller" filename="libgazebo_ros_camera.so">
-					<alwaysOn>true</alwaysOn>
-					<updateRate>30.0</updateRate>
-					<cameraName>virtual_camera</cameraName>
-					<imageTopicName>image_raw</imageTopicName>
-					<cameraInfoTopicName>camera_info</cameraInfoTopicName>
-					<frameName>camera_link</frameName>
-					<hackBaseline>0.07</hackBaseline>
-					<distortionK1>0.0</distortionK1>
-					<distortionK2>0.0</distortionK2>
-					<distortionK3>0.0</distortionK3>
-					<distortionT1>0.0</distortionT1>
-					<distortionT2>0.0</distortionT2>
-				</plugin>
-			</sensor>
-		</gazebo>
+	<link name="projector_link">
+		<visual>
+			<origin xyz="0 0 0" rpy="0 0 0" />
+			<geometry>
+				<box size="0.2 0.1 0.4" />
+			</geometry>
+		</visual>
+		<inertial>
+			<mass value="1" />
+			<origin xyz="0 0 0" />
+			<inertia ixx="0.1" ixy="0.0" ixz="0.0" iyy="0.1" iyz="0.0" izz="0.1" />
+		</inertial>
+	</link>
+	<gazebo>
+		<static>true</static>
+	</gazebo>
+	<gazebo reference="projector_link">
+		<material>Gazebo/Wood</material>
+		<static>true</static>
+		<sensor type="camera" name="virtual_camera">
+			<camera name="projector_head">
+				<horizontal_fov>0.7051310591</horizontal_fov> 				<!-- horizontal field of view in radians -> FOV = 2 arctan(image_width / (2 * focal_lenght)) -->
+				<image>
+					<width>1920</width>
+					<height>1080</height>
+					<format>R8G8B8</format> 								<!-- pixel format -> L8 | R8G8B8 | B8G8R8 | BAYER_RGGB8 | BAYER_BGGR8 | BAYER_GBRG8 | BAYER_GRBG8 -->
+				</image>
+				<clip>
+					<near>0.05</near>
+					<far>25</far>
+				</clip>
+				<noise>
+					<type>gaussian</type>
+					<mean>0.0</mean>
+					<stddev>0.007</stddev>
+				</noise>
+			</camera>
+			<!-- https://github.com/ros-simulation/gazebo_ros_pkgs/blob/hydro-devel/gazebo_plugins/src/gazebo_ros_camera_utils.cpp -->
+			<plugin name="camera_controller" filename="libgazebo_ros_camera.so">
+				<alwaysOn>true</alwaysOn>
+				<updateRate>30.0</updateRate> 								<!-- if 0 -> unlimited -->
+				<cameraName>virtual_camera</cameraName>
+				<imageTopicName>image_raw</imageTopicName>
+				<cameraInfoTopicName>camera_info</cameraInfoTopicName>
+				<frameName>camera_link</frameName>
+				<!-- camera intrinsic parameters -->
+				<CxPrime>0</CxPrime> 										<!-- if 0 - > (image_width + 1) / 2 -->
+				<Cx>0</Cx> 													<!-- if 0 - > (image_width + 1) / 2 -->
+				<Cy>0</Cy> 													<!-- if 0 - > (image_height + 1) / 2 -->
+				<focalLength>0</focalLength> 								<!-- if 0 - > image_width / (2 * tan(HFOV_radians / 2)) -->
+				<hackBaseline>0.07</hackBaseline>
+				<!-- parameters that will be available in future versions of Gazebo -->
+				<distortionK1>0</distortionK1>
+				<distortionK2>0</distortionK2>
+				<distortionK3>0</distortionK3>
+				<distortionT1>0</distortionT1>
+				<distortionT2>0</distortionT2>
+			</plugin>
+		</sensor>
+	</gazebo>
 </robot>
